Commit message: add tip link

File: leg_description/urdf/body.xacro (robot description, xacro)
@@ -23,9 +23,9 @@
 </link>
 <xacro:property name="pi" value="3.1415926" />
-<xacro:leg side="r" num="1" x="0.5" y="-0.19" z="0.022"	angle="-${pi/3}" joint_effort="10000" joint_velocity="100"/>
+<xacro:leg side="r" num="1" x="0.5" y="-0.19" z="0.022"	angle="-${pi/2}" joint_effort="10000" joint_velocity="100"/>
 <xacro:leg side="r" num="2" x="0.0" y="-0.19" z="0.022"	angle="-${pi/2}" joint_effort="10000" joint_velocity="100"/>
-<xacro:leg side="r" num="3" x="-0.5" y="-0.19" z="0.022" angle="-${pi*2/3}" joint_effort="10000" joint_velocity="100"/>
-<xacro:leg side="l" num="1" x="0.5" y="0.19" z="0.022"	angle="${pi/3}" joint_effort="10000" joint_velocity="100"/>
+<xacro:leg side="r" num="3" x="-0.5" y="-0.19" z="0.022" angle="-${pi/2}" joint_effort="10000" joint_velocity="100"/>
+<xacro:leg side="l" num="1" x="0.5" y="0.19" z="0.022"	angle="${pi/2}" joint_effort="10000" joint_velocity="100"/>
 <xacro:leg side="l" num="2" x="0.0" y="0.19" z="0.022"	angle="${pi/2}" joint_effort="10000" joint_velocity="100"/>
-<xacro:leg side="l" num="3" x="-0.5" y="0.19" z="0.022" angle="${pi*2/3}" joint_effort="10000" joint_velocity="100" />
+<xacro:leg side="l" num="3" x="-0.5" y="0.19" z="0.022" angle="${pi/2}" joint_effort="10000" joint_velocity="100" />
 </robot>

File: leg_description/urdf/leg.xacro (robot description, xacro)
@@ -2,5 +2,5 @@
 <robot name="leg" xmlns:xacro="http://www.ros.org/wiki/xacro">
 <xacro:include filename="$(find leg_description)/urdf/materials.xacro" />
-<xacro:include filename="$(find leg_description)/urdf/leg.gazebo" />
+<!-- <xacro:include filename="$(find leg_description)/urdf/leg.gazebo" /> -->
 <xacro:macro name="leg" params="side num x y z angle joint_effort joint_velocity">
 <link name="leg_base_${side}${num}">
@@ -84,5 +84,26 @@
   </collision>
 </link>
-<link name="leg_tip_${side}${num}" />
+<link name="leg_tip_${side}${num}" >
+  <inertial>
+    <origin rpy="0 0 0" xyz="0.09817993031034078 -3.4785017669889708e-06 -0.11373105818820523"/>
+    <mass value="5.477504097726574"/>
+    <inertia ixx="0.062093" ixy="-0.0" ixz="0.023385" iyy="0.070019" iyz="-0.0" izz="0.018221"/>
+  </inertial>
+  <visual>
+    <origin rpy="1.5708 0 0" xyz="0 0 0"/>
+    <geometry>
+        <sphere radius="0.03"/>
+    </geometry>
+    <material name="black"/>
+  </visual>
+  <collision>
+    <origin rpy="1.5708 0 0" xyz="0 0 0"/>
+    <geometry>
+        <sphere radius="0.03"/>
+    </geometry>
+  </collision>
+</link>
+<link name="tip_inter_${side}${num}" />
+<link name="tip_${side}${num}" />
 <joint name="joint_base_link_${side}${num}" type="fixed">
   <origin xyz="${x} ${y} ${z}" rpy="0 0 ${angle}" />
@@ -95,5 +116,5 @@
   <child link="femur_base_${side}${num}"/>
   <axis xyz="0.0 0.0 -1.0"/>
-  <limit lower="-1.5" upper="1.5" effort="${joint_effort}" velocity="${joint_velocity}" />
+  <limit lower="-1.1" upper="1.1" effort="${joint_effort}" velocity="${joint_velocity}" />
 </joint>
 <joint name="joint_femur_${side}${num}" type="revolute">
@@ -111,8 +132,24 @@
   <limit lower="-1.5" upper="0.0" effort="${joint_effort}" velocity="${joint_velocity}" />
 </joint>
-<joint name="tibia_foot_joint_${side}${num}" type="fixed">
-  <origin xyz="0.08 0 -0.40" rpy="0 0 0" />
+<joint name="tibia_foot_joint_${side}${num}" type="revolute">
+  <origin xyz="0.08 0 -0.40" rpy="0 0 -1.57" />
   <parent link="tibia_link_${side}${num}" />
   <child link="leg_tip_${side}${num}" />
+  <axis xyz="1.0 0.0 0.0"/>
+  <limit lower="-3.14" upper="3.14" effort="${joint_effort}" velocity="${joint_velocity}" />
+</joint>
+<joint name="leg_tip_inter_joint_${side}${num}" type="revolute">
+  <origin xyz="0.0 0 -0.0" rpy="0.0 0 0.0" />
+  <parent link="leg_tip_${side}${num}" />
+  <child link="tip_inter_${side}${num}" />
+  <axis xyz="0.0 1.0 0.0"/>
+  <limit lower="-3.14" upper="3.14" effort="${joint_effort}" velocity="${joint_velocity}" />
+</joint>
+<joint name="leg_tip_joint_${side}${num}" type="revolute">
+  <origin xyz="0.0 0 -0.0" rpy="0.0 0 0.0" />
+  <parent link="tip_inter_${side}${num}" />
+  <child link="tip_${side}${num}" />
+  <axis xyz="0.0 0.0 1.0"/>
+  <limit lower="-3.14" upper="3.14" effort="${joint_effort}" velocity="${joint_velocity}" />
 </joint>
 <!-- leg gazebo properties -->
@@ -146,4 +183,10 @@
   <mu1>0.2</mu1>
   <mu2>0.2</mu2>
+  <selfCollide>true</selfCollide>
+</gazebo>
+<gazebo reference="leg_tip_${side}${num}">
+  <material>Gazebo/Black</material>
+  <mu1>1000</mu1>
+  <mu2>1000</mu2>
   <selfCollide>true</selfCollide>
 </gazebo>

Commit message: improves urdf, gazebo controller and IK interface

File: leg_description/urdf/body.xacro (robot description, xacro)
@@ -6,6 +6,7 @@
   <inertial>
     <origin rpy="0 0 0" xyz="0 0 -0.065"/>
-    <mass value="20"/>
-    <inertia ixx="3.251607" ixy="-0.0" ixz="-0.0" iyy="13.028524" iyz="-0.0" izz="16.272836"/>
+    <mass value="5.0"/>
+    <!-- <inertia  ixx="0.7048333333333332" ixy="0" ixz="0" iyy="2.604833333333333" iyz="0" izz="3.3083333333333327" /> -->
+    <inertia  ixx="0.1762083333333333" ixy="0" ixz="0" iyy="0.6512083333333333" iyz="0" izz="0.8270833333333332" />
   </inertial>
   <visual>
@@ -23,9 +24,9 @@
 </link>
 <xacro:property name="pi" value="3.1415926" />
-<xacro:leg side="r" num="1" x="0.5" y="-0.19" z="0.022"	angle="-${pi/2}" joint_effort="10000" joint_velocity="100"/>
-<xacro:leg side="r" num="2" x="0.0" y="-0.19" z="0.022"	angle="-${pi/2}" joint_effort="10000" joint_velocity="100"/>
-<xacro:leg side="r" num="3" x="-0.5" y="-0.19" z="0.022" angle="-${pi/2}" joint_effort="10000" joint_velocity="100"/>
-<xacro:leg side="l" num="1" x="0.5" y="0.19" z="0.022"	angle="${pi/2}" joint_effort="10000" joint_velocity="100"/>
-<xacro:leg side="l" num="2" x="0.0" y="0.19" z="0.022"	angle="${pi/2}" joint_effort="10000" joint_velocity="100"/>
-<xacro:leg side="l" num="3" x="-0.5" y="0.19" z="0.022" angle="${pi/2}" joint_effort="10000" joint_velocity="100" />
+<xacro:leg side="r" num="1" x="0.5" y="-0.19" z="0.022"	angle="-${pi/2}" joint_effort="500" joint_velocity="3.14"/>
+<xacro:leg side="r" num="2" x="0.0" y="-0.19" z="0.022"	angle="-${pi/2}" joint_effort="500" joint_velocity="3.14"/>
+<xacro:leg side="r" num="3" x="-0.5" y="-0.19" z="0.022" angle="-${pi/2}" joint_effort="500" joint_velocity="3.14"/>
+<xacro:leg side="l" num="1" x="0.5" y="0.19" z="0.022"	angle="${pi/2}" joint_effort="500" joint_velocity="3.14"/>
+<xacro:leg side="l" num="2" x="0.0" y="0.19" z="0.022"	angle="${pi/2}" joint_effort="500" joint_velocity="3.14"/>
+<xacro:leg side="l" num="3" x="-0.5" y="0.19" z="0.022" angle="${pi/2}" joint_effort="500" joint_velocity="3.14" />
 </robot>

File: leg_description/urdf/leg.xacro (robot description, xacro)
@@ -8,5 +8,5 @@
     <origin rpy="0 0 0" xyz="-0.004871681061061522 0.00011643429551521872 0.019692846258153093"/>
     <mass value="8.341020253462162"/>
-    <inertia ixx="0.026667" ixy="-2e-05" ixz="-0.000165" iyy="0.028259" iyz="4e-06" izz="0.051461"/>
+    <inertia  ixx="0.03835511729075018" ixy="0" ixz="0" iyy="0.03559944541918172" iyz="0" izz="0.06699597967785346" />
   </inertial>
   <visual>
@@ -28,5 +28,5 @@
     <origin rpy="0 0 0" xyz="0.10872635808676938 0.008582554861478622 0.01963983681426297"/>
     <mass value="5.7419415798639255"/>
-    <inertia ixx="0.009647" ixy="0.004677" ixz="-0.003289" iyy="0.03841" iyz="0.000767" izz="0.04268"/>
+    <inertia  ixx="0.01611425340990051" ixy="0" ixz="0" iyy="0.055107473001172" iyz="0" izz="0.06303439424158978" />
   </inertial>
   <visual>
@@ -48,10 +48,10 @@
     <origin rpy="0 0 0" xyz="0.03630026202441122 7.870816556624017e-05 0.10443637465493055"/>
     <mass value="4.728983887639144"/>
-    <inertia ixx="0.046876" ixy="2.5e-05" ixz="-0.01643" iyy="0.050918" iyz="2.5e-05" izz="0.017083"/>
+    <inertia  ixx="0.008957273120998479" ixy="0" ixz="0" iyy="0.05425147958442127" iyz="0" izz="0.05680332607908645" />
   </inertial>
   <visual>
     <origin rpy="1.5708 -1.045 0" xyz="0 0 0"/>
     <geometry>
-      <mesh filename="package://leg_description/meshes/Femur_Assembly.stl" scale="0.001 0.001 0.001"/>
+      <mesh filename="package://leg_description/meshes/femur_assembly_v2.stl" scale="0.001 0.001 0.001"/>
     </geometry>
     <material name="silver"/>
@@ -60,5 +60,5 @@
     <origin rpy="1.5708 -1.045 0" xyz="0 0 0"/>
     <geometry>
-      <mesh filename="package://leg_description/meshes/Femur_Assembly.stl" scale="0.001 0.001 0.001"/>
+      <mesh filename="package://leg_description/meshes/femur_assembly_v2.stl" scale="0.001 0.001 0.001"/>
     </geometry>
   </collision>
@@ -68,10 +68,10 @@
     <origin rpy="0 0 0" xyz="0.09817993031034078 -3.4785017669889708e-06 -0.11373105818820523"/>
     <mass value="5.477504097726574"/>
-    <inertia ixx="0.062093" ixy="-0.0" ixz="0.023385" iyy="0.070019" iyz="-0.0" izz="0.018221"/>
-  </inertial>
-  <visual>
-    <origin rpy="1.5708 0 0" xyz="0 0 0"/>
-    <geometry>
-      <mesh filename="package://leg_description/meshes/Tibia_Assembly.stl" scale="0.001 0.001 0.001"/>
+    <inertia  ixx="0.08900047312320263" ixy="0" ixz="0" iyy="0.012196295613728567" iyz="0" izz="0.09412713678146542" />
+  </inertial>
+  <visual>
+    <origin rpy="1.5708 0 0" xyz="0 0 0"/>
+    <geometry>
+      <mesh filename="package://leg_description/meshes/tibia_assembly_v2.stl" scale="0.001 0.001 0.001"/>
     </geometry>
     <material name="black"/>
@@ -80,5 +80,25 @@
     <origin rpy="1.5708 0 0" xyz="0 0 0"/>
     <geometry>
-      <mesh filename="package://leg_description/meshes/Tibia_Assembly.stl" scale="0.001 0.001 0.001"/>
+      <mesh filename="package://leg_description/meshes/tibia_assembly_v2.stl" scale="0.001 0.001 0.001"/>
+    </geometry>
+  </collision>
+</link>
+<link name="leg_tip_touch${side}${num}" >
+  <inertial>
+    <origin rpy="0 0 0" xyz="0.09817993031034078 -3.4785017669889708e-06 -0.11373105818820523"/>
+    <mass value="1.0"/>
+    <inertia ixx="0.000006" ixy="-0.0" ixz="0.023385" iyy="0.000006" iyz="-0.0" izz="0.000006"/>
+  </inertial>
+  <visual>
+    <origin rpy="1.5708 0 0" xyz="0 0 0"/>
+    <geometry>
+        <sphere radius="0.03"/>
+    </geometry>
+    <material name="black"/>
+  </visual>
+  <collision>
+    <origin rpy="1.5708 0 0" xyz="0 0 0"/>
+    <geometry>
+        <sphere radius="0.03"/>
     </geometry>
   </collision>
@@ -87,11 +107,11 @@
   <inertial>
     <origin rpy="0 0 0" xyz="0.09817993031034078 -3.4785017669889708e-06 -0.11373105818820523"/>
-    <mass value="5.477504097726574"/>
-    <inertia ixx="0.062093" ixy="-0.0" ixz="0.023385" iyy="0.070019" iyz="-0.0" izz="0.018221"/>
-  </inertial>
-  <visual>
-    <origin rpy="1.5708 0 0" xyz="0 0 0"/>
-    <geometry>
-        <sphere radius="0.03"/>
+    <mass value="0.01"/>
+    <inertia ixx="0.000006" ixy="-0.0" ixz="0.023385" iyy="0.000006" iyz="-0.0" izz="0.000006"/>
+  </inertial>
+  <!-- <visual>
+    <origin rpy="1.5708 0 0" xyz="0 0 0"/>
+    <geometry>
+        <sphere radius="0.003"/>
     </geometry>
     <material name="black"/>
@@ -100,10 +120,22 @@
     <origin rpy="1.5708 0 0" xyz="0 0 0"/>
     <geometry>
-        <sphere radius="0.03"/>
-    </geometry>
-  </collision>
-</link>
-<link name="tip_inter_${side}${num}" />
-<link name="tip_${side}${num}" />
+        <sphere radius="0.003"/>
+    </geometry>
+  </collision> -->
+</link>
+<link name="tip_inter_${side}${num}" >
+  <inertial>
+    <origin rpy="0 0 0" xyz="0.09817993031034078 -3.4785017669889708e-06 -0.11373105818820523"/>
+    <mass value="0.01"/>
+    <inertia ixx="0.000006" ixy="-0.0" ixz="0.023385" iyy="0.000006" iyz="-0.0" izz="0.000006"/>
+  </inertial>
+</link>
+<link name="tip_${side}${num}" >
+  <inertial>
+    <origin rpy="0 0 0" xyz="0.09817993031034078 -3.4785017669889708e-06 -0.11373105818820523"/>
+    <mass value="0.01"/>
+    <inertia ixx="0.000006" ixy="-0.0" ixz="0.023385" iyy="0.000006" iyz="-0.0" izz="0.000006"/>
+  </inertial>
+</link>
 <joint name="joint_base_link_${side}${num}" type="fixed">
   <origin xyz="${x} ${y} ${z}" rpy="0 0 ${angle}" />
@@ -132,4 +164,9 @@
   <limit lower="-1.5" upper="0.0" effort="${joint_effort}" velocity="${joint_velocity}" />
 </joint>
+<joint name="tibia_foot_touch_joint_${side}${num}" type="fixed">
+  <origin xyz="0.08 0 -0.40" rpy="0 0 -1.57" />
+  <parent link="tibia_link_${side}${num}" />
+  <child link="leg_tip_touch${side}${num}" />
+</joint>
 <joint name="tibia_foot_joint_${side}${num}" type="revolute">
   <origin xyz="0.08 0 -0.40" rpy="0 0 -1.57" />
@@ -137,5 +174,5 @@
   <child link="leg_tip_${side}${num}" />
   <axis xyz="1.0 0.0 0.0"/>
-  <limit lower="-3.14" upper="3.14" effort="${joint_effort}" velocity="${joint_velocity}" />
+  <limit lower="-3.14" upper="3.14" effort="0.0" velocity="0.0" />
 </joint>
 <joint name="leg_tip_inter_joint_${side}${num}" type="revolute">
@@ -144,5 +181,5 @@
   <child link="tip_inter_${side}${num}" />
   <axis xyz="0.0 1.0 0.0"/>
-  <limit lower="-3.14" upper="3.14" effort="${joint_effort}" velocity="${joint_velocity}" />
+  <limit lower="-3.14" upper="3.14" effort="0.0" velocity="0.0" />
 </joint>
 <joint name="leg_tip_joint_${side}${num}" type="revolute">
@@ -151,43 +188,75 @@
   <child link="tip_${side}${num}" />
   <axis xyz="0.0 0.0 1.0"/>
-  <limit lower="-3.14" upper="3.14" effort="${joint_effort}" velocity="${joint_velocity}" />
+  <limit lower="-3.14" upper="3.14" effort="0.0" velocity="0.0" />
 </joint>
 <!-- leg gazebo properties -->
 <gazebo reference="base_link">
   <material>Gazebo/Red</material>
-  <mu1>0.2</mu1>
-  <mu2>0.2</mu2>
-  <selfCollide>true</selfCollide>
-  <gravity>true</gravity>
+  <!-- <mu1>0.2</mu1> -->
+  <!-- <mu2>0.2</mu2> -->
+  <!-- <selfCollide>false</selfCollide> -->
+  <!-- <gravity>true</gravity> -->
 </gazebo>
 <gazebo reference="leg_base_${side}${num}">
   <material>Gazebo/White</material>
-  <mu1>0.2</mu1>
+  <!-- <mu1>0.2</mu1>
   <mu2>0.2</mu2>
-  <selfCollide>true</selfCollide>
+  <selfCollide>false</selfCollide> -->
 </gazebo>
 <gazebo reference="femur_base_${side}${num}">
   <material>Gazebo/Black</material>
-  <mu1>0.2</mu1>
+  <!-- <mu1>0.2</mu1>
   <mu2>0.2</mu2>
-  <selfCollide>true</selfCollide>
+  <selfCollide>false</selfCollide> -->
 </gazebo>
 <gazebo reference="femur_link_${side}${num}">
   <material>Gazebo/White</material>
-  <mu1>0.2</mu1>
+  <!-- <mu1>0.2</mu1>
   <mu2>0.2</mu2>
-  <selfCollide>true</selfCollide>
+  <selfCollide>false</selfCollide> -->
 </gazebo>
 <gazebo reference="tibia_link_${side}${num}">
   <material>Gazebo/Black</material>
-  <mu1>0.2</mu1>
+  <!-- <mu1>0.2</mu1>
   <mu2>0.2</mu2>
-  <selfCollide>true</selfCollide>
+  <selfCollide>false</selfCollide> -->
+</gazebo>
+<gazebo reference="leg_tip_touch${side}${num}">
+  <!-- <kp>10.0</kp>
+  <kd>0.01</kd> -->
+  <mu>0.90</mu>
+  <mu1>0.90</mu1>
+  <mu2>0.90</mu2>
+  <maxVel>0.0</maxVel>
+  <!-- <minDepth>0.001</minDepth> -->
+  <material>Gazebo/FlatBlack</material>
+  <selfCollide>false</selfCollide>
 </gazebo>
 <gazebo reference="leg_tip_${side}${num}">
-  <material>Gazebo/Black</material>
-  <mu1>1000</mu1>
-  <mu2>1000</mu2>
-  <selfCollide>true</selfCollide>
+  <!-- <kp>1000000.0</kp>
+  <kd>1.0</kd>
+  <mu1>1000000.0</mu1>
+  <mu2>1000000.0</mu2>
+  <maxVel>0.0</maxVel>
+  <minDepth>0.001</minDepth> -->
+  <material>Gazebo/FlatBlack</material>
+</gazebo>
+<gazebo reference="tip_inter_${side}${num}">
+  <!-- <kp>1000000.0</kp>
+  <kd>1.0</kd>
+  <mu1>100.0</mu1>
+  <mu2>100.0</mu2>
+  <maxVel>0.0</maxVel>
+  <minDepth>0.001</minDepth> -->
+  <material>Gazebo/FlatBlack</material>
+</gazebo>
+<gazebo reference="tip_${side}${num}">
+  <!-- <kp>1000000.0</kp>
+  <kd>1.0</kd>
+  <mu1>0.8</mu1>
+  <mu2>0.8</mu2>
+  <maxVel>0.0</maxVel>
+  <minDepth>0.001</minDepth> -->
+  <material>Gazebo/FlatBlack</material>
 </gazebo>
 <!-- Leg transmission properties  -->
@@ -195,8 +264,8 @@
   <type>transmission_interface/SimpleTransmission</type>
   <joint name="joint_base_${side}${num}">
-    <hardwareInterface>hardware_interface/EffortJointInterface</hardwareInterface>
+    <hardwareInterface>hardware_interface/PositionJointInterface</hardwareInterface>
   </joint>
   <actuator name="joint_base_${side}${num}_actr">
-    <hardwareInterface>hardware_interface/EffortJointInterface</hardwareInterface>
+    <hardwareInterface>hardware_interface/PositionJointInterface</hardwareInterface>
     <mechanicalReduction>1</mechanicalReduction>
   </actuator>
@@ -205,8 +274,8 @@
   <type>transmission_interface/SimpleTransmission</type>
   <joint name="joint_femur_${side}${num}">
-    <hardwareInterface>hardware_interface/EffortJointInterface</hardwareInterface>
+    <hardwareInterface>hardware_interface/PositionJointInterface</hardwareInterface>
   </joint>
   <actuator name="joint_femur_${side}${num}_actr">
-    <hardwareInterface>hardware_interface/EffortJointInterface</hardwareInterface>
+    <hardwareInterface>hardware_interface/PositionJointInterface</hardwareInterface>
     <mechanicalReduction>1</mechanicalReduction>
   </actuator>
@@ -215,8 +284,38 @@
   <type>transmission_interface/SimpleTransmission</type>
   <joint name="joint_tibia_${side}${num}">
-    <hardwareInterface>hardware_interface/EffortJointInterface</hardwareInterface>
+    <hardwareInterface>hardware_interface/PositionJointInterface</hardwareInterface>
   </joint>
   <actuator name="joint_tibia_${side}${num}_actr">
-    <hardwareInterface>hardware_interface/EffortJointInterface</hardwareInterface>
+    <hardwareInterface>hardware_interface/PositionJointInterface</hardwareInterface>
+    <mechanicalReduction>1</mechanicalReduction>
+  </actuator>
+</transmission>
+<transmission name="tibia_foot_joint_${side}${num}_tran">
+  <type>transmission_interface/SimpleTransmission</type>
+  <joint name="tibia_foot_joint_${side}${num}">
+    <hardwareInterface>hardware_interface/PositionJointInterface</hardwareInterface>
+  </joint>
+  <actuator name="tibia_foot_joint_${side}${num}_actr">
+    <hardwareInterface>hardware_interface/PositionJointInterface</hardwareInterface>
+    <mechanicalReduction>1</mechanicalReduction>
+  </actuator>
+</transmission>
+<transmission name="leg_tip_inter_joint_${side}${num}_tran">
+  <type>transmission_interface/SimpleTransmission</type>
+  <joint name="leg_tip_inter_joint_${side}${num}">
+    <hardwareInterface>hardware_interface/PositionJointInterface</hardwareInterface>
+  </joint>
+  <actuator name="leg_tip_inter_joint_${side}${num}_actr">
+    <hardwareInterface>hardware_interface/PositionJointInterface</hardwareInterface>
+    <mechanicalReduction>1</mechanicalReduction>
+  </actuator>
+</transmission>
+<transmission name="leg_tip_joint_${side}${num}_tran">
+  <type>transmission_interface/SimpleTransmission</type>
+  <joint name="leg_tip_joint_${side}${num}">
+    <hardwareInterface>hardware_interface/PositionJointInterface</hardwareInterface>
+  </joint>
+  <actuator name="leg_tip_joint_${side}${num}_actr">
+    <hardwareInterface>hardware_interface/PositionJointInterface</hardwareInterface>
     <mechanicalReduction>1</mechanicalReduction>
   </actuator>
