Commit message: tune effort joint controller

File: leg_description/urdf/body.xacro (robot description, xacro)
@@ -7,5 +7,4 @@
     <origin rpy="0 0 0" xyz="0 0 -0.065"/>
     <mass value="5.0"/>
-    <!-- <inertia  ixx="0.7048333333333332" ixy="0" ixz="0" iyy="2.604833333333333" iyz="0" izz="3.3083333333333327" /> -->
     <inertia  ixx="0.1762083333333333" ixy="0" ixz="0" iyy="0.6512083333333333" iyz="0" izz="0.8270833333333332" />
   </inertial>
@@ -24,9 +23,9 @@
 </link>
 <xacro:property name="pi" value="3.1415926" />
-<xacro:leg side="r" num="1" x="0.5" y="-0.19" z="0.022"	angle="-${pi/2}" joint_effort="500" joint_velocity="3.14"/>
-<xacro:leg side="r" num="2" x="0.0" y="-0.19" z="0.022"	angle="-${pi/2}" joint_effort="500" joint_velocity="3.14"/>
-<xacro:leg side="r" num="3" x="-0.5" y="-0.19" z="0.022" angle="-${pi/2}" joint_effort="500" joint_velocity="3.14"/>
-<xacro:leg side="l" num="1" x="0.5" y="0.19" z="0.022"	angle="${pi/2}" joint_effort="500" joint_velocity="3.14"/>
-<xacro:leg side="l" num="2" x="0.0" y="0.19" z="0.022"	angle="${pi/2}" joint_effort="500" joint_velocity="3.14"/>
-<xacro:leg side="l" num="3" x="-0.5" y="0.19" z="0.022" angle="${pi/2}" joint_effort="500" joint_velocity="3.14" />
+<xacro:leg side="r" num="1" x="0.5" y="-0.19" z="0.022"	angle="-${pi/2}" joint_effort="200.0" joint_velocity="3.14"/>
+<xacro:leg side="r" num="2" x="0.0" y="-0.19" z="0.022"	angle="-${pi/2}" joint_effort="200.0" joint_velocity="3.14"/>
+<xacro:leg side="r" num="3" x="-0.5" y="-0.19" z="0.022" angle="-${pi/2}" joint_effort="200.0" joint_velocity="3.14"/>
+<xacro:leg side="l" num="1" x="0.5" y="0.19" z="0.022"	angle="${pi/2}" joint_effort="200.0" joint_velocity="3.14"/>
+<xacro:leg side="l" num="2" x="0.0" y="0.19" z="0.022"	angle="${pi/2}" joint_effort="200.0" joint_velocity="3.14"/>
+<xacro:leg side="l" num="3" x="-0.5" y="0.19" z="0.022" angle="${pi/2}" joint_effort="200.0" joint_velocity="3.14" />
 </robot>

File: leg_description/urdf/leg.xacro (robot description, xacro)
@@ -7,6 +7,6 @@
   <inertial>
     <origin rpy="0 0 0" xyz="-0.004871681061061522 0.00011643429551521872 0.019692846258153093"/>
-    <mass value="8.341020253462162"/>
-    <inertia  ixx="0.03835511729075018" ixy="0" ixz="0" iyy="0.03559944541918172" iyz="0" izz="0.06699597967785346" />
+    <mass value="1.0"/>
+    <inertia  ixx="0.004598372396330038" ixy="0" ixz="0" iyy="0.004267996520498223" iyz="0" izz="0.008032108500161596" />
   </inertial>
   <visual>
@@ -27,6 +27,6 @@
   <inertial>
     <origin rpy="0 0 0" xyz="0.10872635808676938 0.008582554861478622 0.01963983681426297"/>
-    <mass value="5.7419415798639255"/>
-    <inertia  ixx="0.01611425340990051" ixy="0" ixz="0" iyy="0.055107473001172" iyz="0" izz="0.06303439424158978" />
+    <mass value="1.0"/>
+    <inertia  ixx="0.0028064119402417174" ixy="0" ixz="0" iyy="0.00959735870431443" iyz="0" izz="0.010977888465922635" />
   </inertial>
   <visual>
@@ -47,6 +47,6 @@
   <inertial>
     <origin rpy="0 0 0" xyz="0.03630026202441122 7.870816556624017e-05 0.10443637465493055"/>
-    <mass value="4.728983887639144"/>
-    <inertia  ixx="0.008957273120998479" ixy="0" ixz="0" iyy="0.05425147958442127" iyz="0" izz="0.05680332607908645" />
+    <mass value="3.0"/>
+    <inertia  ixx="0.005681961724590655" ixy="0" ixz="0" iyy="0.03441321342556238" iyz="0" izz="0.036031663762595055" />
   </inertial>
   <visual>
@@ -67,6 +67,6 @@
   <inertial>
     <origin rpy="0 0 0" xyz="0.09817993031034078 -3.4785017669889708e-06 -0.11373105818820523"/>
-    <mass value="5.477504097726574"/>
-    <inertia  ixx="0.08900047312320263" ixy="0" ixz="0" iyy="0.012196295613728567" iyz="0" izz="0.09412713678146542" />
+    <mass value="2.5"/>
+    <inertia  ixx="0.04686563322871321" ixy="0" ixz="0" iyy="0.005565338161944915" iyz="0" izz="0.04920430472399146" />
   </inertial>
   <visual>
@@ -87,11 +87,31 @@
   <inertial>
     <origin rpy="0 0 0" xyz="0.09817993031034078 -3.4785017669889708e-06 -0.11373105818820523"/>
-    <mass value="1.0"/>
+    <mass value="0.001"/>
+    <inertia ixx="0.000006" ixy="-0.0" ixz="0.00023385" iyy="0.000006" iyz="-0.0" izz="0.000006"/>
+  </inertial>
+  <!-- <visual>
+    <origin rpy="1.5708 0 0" xyz="0 0 0"/>
+    <geometry>
+        <sphere radius="0.03"/>
+    </geometry>
+    <material name="black"/>
+  </visual>
+  <collision>
+    <origin rpy="1.5708 0 0" xyz="0 0 0"/>
+    <geometry>
+        <sphere radius="0.03"/>
+    </geometry>
+  </collision> -->
+</link>
+<link name="leg_tip_${side}${num}" >
+  <inertial>
+    <origin rpy="0 0 0" xyz="0.09817993031034078 -3.4785017669889708e-06 -0.11373105818820523"/>
+    <mass value="0.001"/>
     <inertia ixx="0.000006" ixy="-0.0" ixz="0.023385" iyy="0.000006" iyz="-0.0" izz="0.000006"/>
   </inertial>
-  <visual>
-    <origin rpy="1.5708 0 0" xyz="0 0 0"/>
-    <geometry>
-        <sphere radius="0.03"/>
+  <!-- <visual>
+    <origin rpy="1.5708 0 0" xyz="0 0 0"/>
+    <geometry>
+        <sphere radius="0.003"/>
     </geometry>
     <material name="black"/>
@@ -100,39 +120,19 @@
     <origin rpy="1.5708 0 0" xyz="0 0 0"/>
     <geometry>
-        <sphere radius="0.03"/>
-    </geometry>
-  </collision>
-</link>
-<link name="leg_tip_${side}${num}" >
-  <inertial>
-    <origin rpy="0 0 0" xyz="0.09817993031034078 -3.4785017669889708e-06 -0.11373105818820523"/>
-    <mass value="0.01"/>
+        <sphere radius="0.003"/>
+    </geometry>
+  </collision> -->
+</link>
+<link name="tip_inter_${side}${num}" >
+  <inertial>
+    <origin rpy="0 0 0" xyz="0.09817993031034078 -3.4785017669889708e-06 -0.11373105818820523"/>
+    <mass value="0.001"/>
     <inertia ixx="0.000006" ixy="-0.0" ixz="0.023385" iyy="0.000006" iyz="-0.0" izz="0.000006"/>
   </inertial>
-  <!-- <visual>
-    <origin rpy="1.5708 0 0" xyz="0 0 0"/>
-    <geometry>
-        <sphere radius="0.003"/>
-    </geometry>
-    <material name="black"/>
-  </visual>
-  <collision>
-    <origin rpy="1.5708 0 0" xyz="0 0 0"/>
-    <geometry>
-        <sphere radius="0.003"/>
-    </geometry>
-  </collision> -->
-</link>
-<link name="tip_inter_${side}${num}" >
-  <inertial>
-    <origin rpy="0 0 0" xyz="0.09817993031034078 -3.4785017669889708e-06 -0.11373105818820523"/>
-    <mass value="0.01"/>
-    <inertia ixx="0.000006" ixy="-0.0" ixz="0.023385" iyy="0.000006" iyz="-0.0" izz="0.000006"/>
-  </inertial>
 </link>
 <link name="tip_${side}${num}" >
   <inertial>
     <origin rpy="0 0 0" xyz="0.09817993031034078 -3.4785017669889708e-06 -0.11373105818820523"/>
-    <mass value="0.01"/>
+    <mass value="0.001"/>
     <inertia ixx="0.000006" ixy="-0.0" ixz="0.023385" iyy="0.000006" iyz="-0.0" izz="0.000006"/>
   </inertial>
@@ -195,4 +195,5 @@
   <!-- <mu1>0.2</mu1> -->
   <!-- <mu2>0.2</mu2> -->
+  <!-- <maxVel>0.000000</maxVel> -->
   <!-- <selfCollide>false</selfCollide> -->
   <!-- <gravity>true</gravity> -->
@@ -201,4 +202,5 @@
   <material>Gazebo/White</material>
   <!-- <mu1>0.2</mu1>
+  <maxVel>0.000000</maxVel>
   <mu2>0.2</mu2>
   <selfCollide>false</selfCollide> -->
@@ -207,4 +209,5 @@
   <material>Gazebo/Black</material>
   <!-- <mu1>0.2</mu1>
+  <maxVel>0.000000</maxVel>
   <mu2>0.2</mu2>
   <selfCollide>false</selfCollide> -->
@@ -214,22 +217,29 @@
   <!-- <mu1>0.2</mu1>
   <mu2>0.2</mu2>
+  <maxVel>0.000000</maxVel>
   <selfCollide>false</selfCollide> -->
 </gazebo>
 <gazebo reference="tibia_link_${side}${num}">
-  <material>Gazebo/Black</material>
-  <!-- <mu1>0.2</mu1>
-  <mu2>0.2</mu2>
-  <selfCollide>false</selfCollide> -->
+  <material>Gazebo/FlatBlack</material>
+  <!-- <gravity>true</gravity> -->
+  <!-- <dampingFactor>0.003</dampingFactor>  -->
+  <maxVel>0.0</maxVel>
+  <minDepth>0.001</minDepth>
+  <!-- <mu1>100000.0</mu1> -->
+  <!-- <mu2>100000.0</mu2> -->
+  <!-- <fdir1>1 0 0</fdir1> -->
+  <kp>1000000.0</kp>
+  <kd>1.0</kd>
+  <!-- <selfCollide>false</selfCollide> -->
+  <!-- <maxContacts> 10 </maxContacts> -->
+  <!-- <kp>1000000.0</kp>     -->
+  <!-- <kd>10.0</kd>     -->
+  <mu1>0.8</mu1>
+  <mu2>0.8</mu2>
 </gazebo>
 <gazebo reference="leg_tip_touch${side}${num}">
   <!-- <kp>10.0</kp>
   <kd>0.01</kd> -->
-  <mu>0.90</mu>
-  <mu1>0.90</mu1>
-  <mu2>0.90</mu2>
-  <maxVel>0.0</maxVel>
-  <!-- <minDepth>0.001</minDepth> -->
-  <material>Gazebo/FlatBlack</material>
-  <selfCollide>false</selfCollide>
+  <!-- <maxVel>0.000000</maxVel> -->
 </gazebo>
 <gazebo reference="leg_tip_${side}${num}">
@@ -240,4 +250,5 @@
   <maxVel>0.0</maxVel>
   <minDepth>0.001</minDepth> -->
+  <!-- <maxVel>0.000000</maxVel> -->
   <material>Gazebo/FlatBlack</material>
 </gazebo>
@@ -249,4 +260,5 @@
   <maxVel>0.0</maxVel>
   <minDepth>0.001</minDepth> -->
+  <!-- <maxVel>0.000000</maxVel> -->
   <material>Gazebo/FlatBlack</material>
 </gazebo>
@@ -258,4 +270,5 @@
   <maxVel>0.0</maxVel>
   <minDepth>0.001</minDepth> -->
+  <!-- <maxVel>0.000000</maxVel> -->
   <material>Gazebo/FlatBlack</material>
 </gazebo>
@@ -264,8 +277,8 @@
   <type>transmission_interface/SimpleTransmission</type>
   <joint name="joint_base_${side}${num}">
-    <hardwareInterface>hardware_interface/PositionJointInterface</hardwareInterface>
+    <hardwareInterface>hardware_interface/EffortJointInterface</hardwareInterface>
   </joint>
   <actuator name="joint_base_${side}${num}_actr">
-    <hardwareInterface>hardware_interface/PositionJointInterface</hardwareInterface>
+    <hardwareInterface>hardware_interface/EffortJointInterface</hardwareInterface>
     <mechanicalReduction>1</mechanicalReduction>
   </actuator>
@@ -274,8 +287,8 @@
   <type>transmission_interface/SimpleTransmission</type>
   <joint name="joint_femur_${side}${num}">
-    <hardwareInterface>hardware_interface/PositionJointInterface</hardwareInterface>
+    <hardwareInterface>hardware_interface/EffortJointInterface</hardwareInterface>
   </joint>
   <actuator name="joint_femur_${side}${num}_actr">
-    <hardwareInterface>hardware_interface/PositionJointInterface</hardwareInterface>
+    <hardwareInterface>hardware_interface/EffortJointInterface</hardwareInterface>
     <mechanicalReduction>1</mechanicalReduction>
   </actuator>
@@ -284,8 +297,8 @@
   <type>transmission_interface/SimpleTransmission</type>
   <joint name="joint_tibia_${side}${num}">
-    <hardwareInterface>hardware_interface/PositionJointInterface</hardwareInterface>
+    <hardwareInterface>hardware_interface/EffortJointInterface</hardwareInterface>
   </joint>
   <actuator name="joint_tibia_${side}${num}_actr">
-    <hardwareInterface>hardware_interface/PositionJointInterface</hardwareInterface>
+    <hardwareInterface>hardware_interface/EffortJointInterface</hardwareInterface>
     <mechanicalReduction>1</mechanicalReduction>
   </actuator>
@@ -294,8 +307,8 @@
   <type>transmission_interface/SimpleTransmission</type>
   <joint name="tibia_foot_joint_${side}${num}">
-    <hardwareInterface>hardware_interface/PositionJointInterface</hardwareInterface>
+    <hardwareInterface>hardware_interface/EffortJointInterface</hardwareInterface>
   </joint>
   <actuator name="tibia_foot_joint_${side}${num}_actr">
-    <hardwareInterface>hardware_interface/PositionJointInterface</hardwareInterface>
+    <hardwareInterface>hardware_interface/EffortJointInterface</hardwareInterface>
     <mechanicalReduction>1</mechanicalReduction>
   </actuator>
@@ -304,8 +317,8 @@
   <type>transmission_interface/SimpleTransmission</type>
   <joint name="leg_tip_inter_joint_${side}${num}">
-    <hardwareInterface>hardware_interface/PositionJointInterface</hardwareInterface>
+    <hardwareInterface>hardware_interface/EffortJointInterface</hardwareInterface>
   </joint>
   <actuator name="leg_tip_inter_joint_${side}${num}_actr">
-    <hardwareInterface>hardware_interface/PositionJointInterface</hardwareInterface>
+    <hardwareInterface>hardware_interface/EffortJointInterface</hardwareInterface>
     <mechanicalReduction>1</mechanicalReduction>
   </actuator>
@@ -314,8 +327,8 @@
   <type>transmission_interface/SimpleTransmission</type>
   <joint name="leg_tip_joint_${side}${num}">
-    <hardwareInterface>hardware_interface/PositionJointInterface</hardwareInterface>
+    <hardwareInterface>hardware_interface/EffortJointInterface</hardwareInterface>
   </joint>
   <actuator name="leg_tip_joint_${side}${num}_actr">
-    <hardwareInterface>hardware_interface/PositionJointInterface</hardwareInterface>
+    <hardwareInterface>hardware_interface/EffortJointInterface</hardwareInterface>
     <mechanicalReduction>1</mechanicalReduction>
   </actuator>

Commit message: feat(leg_description): migrate to ROS 2 Jazzy, update package format, and add display.launch.py

File: leg_description/urdf/body.xacro (robot description, xacro)
@@ -22,10 +22,9 @@
   </collision>
 </link>
-<xacro:property name="pi" value="3.1415926" />
 <xacro:leg side="r" num="1" x="0.5" y="-0.19" z="0.022"	angle="-${pi/2}" joint_effort="10000.0" joint_velocity="1.57"/>
 <xacro:leg side="r" num="2" x="0.0" y="-0.19" z="0.022"	angle="-${pi/2}" joint_effort="10000.0" joint_velocity="1.57"/>
 <xacro:leg side="r" num="3" x="-0.5" y="-0.19" z="0.022" angle="-${pi/2}" joint_effort="10000.0" joint_velocity="1.57"/>
-<xacro:leg side="l" num="1" x="0.5" y="0.19" z="0.022"	angle="${pi/2}" joint_effort="10000.0" joint_velocity="1.57"/>
-<xacro:leg side="l" num="2" x="0.0" y="0.19" z="0.022"	angle="${pi/2}" joint_effort="10000.0" joint_velocity="1.57"/>
-<xacro:leg side="l" num="3" x="-0.5" y="0.19" z="0.022" angle="${pi/2}" joint_effort="10000.0" joint_velocity="1.57" />
+<xacro:leg side="l" num="1" x="0.5" y="0.19" z="0.022"	angle="${3.1415926/2}" joint_effort="10000.0" joint_velocity="1.57"/>
+<xacro:leg side="l" num="2" x="0.0" y="0.19" z="0.022"	angle="${3.1415926/2}" joint_effort="10000.0" joint_velocity="1.57"/>
+<xacro:leg side="l" num="3" x="-0.5" y="0.19" z="0.022" angle="${3.1415926/2}" joint_effort="10000.0" joint_velocity="1.57" />
 </robot>
